Commit message: [fix] up gazebo

File: gazebo_mbot_go_maze/urdf/mbot_base.xacro (robot description, xacro)
@@ -154,5 +154,5 @@
   </xacro:macro>
   <xacro:macro name="caster" params="prefix reflect">
-    <joint name="${prefix}_caster_joint" type="continuous">
+    <joint name="${prefix}_caster_joint" type="fixed">
       <origin xyz="${reflect*caster_joint_x} ${caster_joint_y} ${-caster_joint_z}" rpy="0 0 0" />
       <parent link="base_link"/>
@@ -190,23 +190,25 @@
         <plugin name="differential_drive_controller"
                 filename="libgazebo_ros_diff_drive.so">
-            <rosDebugLevel>Debug</rosDebugLevel>
-            <publishWheelTF>true</publishWheelTF>
-            <robotNamespace>/</robotNamespace>
-            <publishTf>1</publishTf>
-            <publishWheelJointState>true</publishWheelJointState>
-            <alwaysOn>true</alwaysOn>
-            <updateRate>100.0</updateRate>
-            <legacyMode>true</legacyMode>
+            <ros_debug_level>Debug</ros_debug_level>
+            <robot_namespace>/</robot_namespace>
+            <publish_tf>1</publish_tf>
+            <publish_wheel_joint_state>true</publish_wheel_joint_state>
+            <always_on>true</always_on>
+            <update_rate>100.0</update_rate>
+            <legacy_mode>true</legacy_mode>
             <left_joint>left_wheel_joint</left_joint>
             <right_joint>right_wheel_joint</right_joint>
             <wheel_separation>${wheel_joint_y*2}</wheel_separation>
             <wheel_diameter>${2*wheel_radius}</wheel_diameter>
-            <broadcastTF>1</broadcastTF>
-            <wheelTorque>30</wheelTorque>
-            <wheelAcceleration>1.8</wheelAcceleration>
-            <commandTopic>cmd_vel</commandTopic>
-            <odometryFrame>odom</odometryFrame>
-            <odometryTopic>odom</odometryTopic>
-            <robotBaseFrame>base_footprint</robotBaseFrame>
+            <broadcast_TF>1</broadcast_TF>
+            <max_wheel_torque>30</max_wheel_torque>
+            <max_wheel_acceleration>1.8</max_wheel_acceleration>
+            <command_topic>cmd_vel</command_topic>
+            <odometry_frame>odom</odometry_frame>
+            <odometry_topic>odom</odometry_topic>
+            <robot_base_frame>base_footprint</robot_base_frame>
+            <publish_odom>true</publish_odom>
+            <publish_odom_tf>true</publish_odom_tf>
+            <publish_wheel_tf>true</publish_wheel_tf>
         </plugin>
     </gazebo>

File: gazebo_mbot_go_maze/urdf/sensor/camera.xacro (robot description, xacro)
@@ -53,11 +53,11 @@
             </camera>
             <plugin name="gazebo_camera_${prefix}" filename="libgazebo_ros_camera.so">
-                <alwaysOn>true</alwaysOn>
-                <updateRate>0.0</updateRate>
-                <cameraName>/camera_${prefix}</cameraName>
-                <imageTopicName>image_raw</imageTopicName>
-                <cameraInfoTopicName>camera_info</cameraInfoTopicName>
-                <frameName>${prefix}_camera_link</frameName>
-                <hackBaseline>0.07</hackBaseline>
+                <always_on>true</always_on>
+                <update_rate>0.0</update_rate>
+                <camera_name>/camera_${prefix}</camera_name>
+                <image_topic_name>image_raw</image_topic_name>
+                <camera_info_topic_name>camera_info</camera_info_topic_name>
+                <frame_name>${prefix}_camera_link</frame_name>
+                <hack_baseline>0.07</hack_baseline>
                 <distortionK1>0.0</distortionK1>
                 <distortionK2>0.0</distortionK2>

File: gazebo_mbot_go_maze/urdf/sensor/laser.xacro (robot description, xacro)
@@ -57,7 +57,10 @@
                 </noise>
             </ray>
-            <plugin name="gazebo_rplidar" filename="libgazebo_ros_laser.so">
-                <topicName>/scan</topicName>
-                <frameName>laser_link</frameName>
+            <plugin name="gazebo_rplidar" filename="libgazebo_ros_ray_sensor.so">
+              <ros>
+                <namespace>/</namespace>
+                <remapping>~/out:=scan</remapping>
+              </ros>
+              <output_type>sensor_msgs/LaserScan</output_type>
             </plugin>
         </sensor>

Commit message: [fix] up it

File: gazebo_mbot_go_maze/urdf/mbot_base.xacro (robot description, xacro)
@@ -154,5 +154,5 @@
   </xacro:macro>
   <xacro:macro name="caster" params="prefix reflect">
-    <joint name="${prefix}_caster_joint" type="fixed">
+    <joint name="${prefix}_caster_joint" type="continuous">
       <origin xyz="${reflect*caster_joint_x} ${caster_joint_y} ${-caster_joint_z}" rpy="0 0 0" />
       <parent link="base_link"/>
@@ -184,6 +184,7 @@
     <xacro:wheel prefix="left"  reflect="1"/>
     <xacro:wheel prefix="right"  reflect="-1"/>
-    <xacro:caster prefix="front"  reflect="1"/>
-    <xacro:caster prefix="back"  reflect="-1"/>
+    <!-- TODO: caster can not work , so delete it ! -->
+    <!-- <xacro:caster prefix="front"  reflect="1"/>
+    <xacro:caster prefix="back"  reflect="-1"/>   -->
     <!-- controller -->
     <gazebo>
